File: Git_Tutorial.kicad_sch (KiCad schematic)
At the start: 0 parts

Commit message: addedname2
Other:
- note added: "Margaret New name!"
Changed lines of the file:
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@@
+		)
+	)
+	(text "Margaret New name!"
+		(exclude_from_sim no)
+		(at 56.515 123.19 0)
+		(effects
+			(font
+				(size 1.27 1.27)
+			)
 		)
 	)
