File: Git_Tutorial.kicad_sch (KiCad schematic)
At the start: 0 parts

Commit message: cleared
Other:
- note removed: "Luke Scholler"
- note removed: "new brnach test"
Changed lines of the file:
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@@
-		)
-	)
-	(text "Luke Scholler"
-		(exclude_from_sim no)
-		(at 229.616 32.512 0)
-		(effects
-			(font
-				(size 1.27 1.27)
-			)
-		)
-	)
-	(text "new brnach test\n"
-		(exclude_from_sim no)
-		(at 87.884 138.43 0)
-		(effects
-			(font
-				(size 1.27 1.27)
-			)
 		)
 	)

Commit message: added heather name
Other:
- note added: "Heather Schwartz"
Changed lines of the file:
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@@
+		)
+	)
+	(text "Heather Schwartz"
+		(exclude_from_sim no)
+		(at 48.26 114.3 0)
+		(effects
+			(font
+				(size 1.27 1.27)
+			)
 		)
 	)

Commit message: added heather name round 2
Other:
- note added: "Margaret Mei"
Changed lines of the file:
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@@
 (kicad_sch
-	(version 20250114)
+	(version 20260306)
 	(generator "eeschema")
-	(generator_version "9.0")
+	(generator_version "10.0")
 	(paper "A4")
+	(text "Margaret Mei"
+		(exclude_from_sim no)
+		(at 57.785 114.3 0)
+		(effects
+			(font
+				(size 1.27 1.27)
+			)
+		)
+	)
 	(text "Steps to make a contribution:\n\n1. insert a sheet: place -> add sheet\n	a. Rename the sheet to whatever you want and MATCH THE NAME TO THE SHEET FILE NAME\n\n2. Add anything within the sheet\n\n3. Save and follow the instructions on github to push"
 		(exclude_from_sim no)
@@
 	(text "Heather Schwartz"
 		(exclude_from_sim no)
-		(at 48.26 114.3 0)
+		(at 135.89 108.204 0)
 		(effects
 			(font
@@
 		)
 		(fill
-			(color 0 0 0 0.0000)
+			(color 0 0 0 0)
 		)
 		(property "Sheetname" "Example_sheet"
 			(at 137.16 74.2184 0)
+			(show_name no)
+			(do_not_autoplace no)
 			(effects
 				(font
@@
 		(property "Sheetfile" "example_sheet.kicad_sch"
 			(at 137.16 90.7546 0)
+			(show_name no)
+			(do_not_autoplace no)
 			(effects
 				(font
