File: example_sheet.kicad_sch (KiCad schematic)
At the start: 5 parts, among them J1 Conn_Coaxial, J2 Conn_Coaxial

Commit message: cleared
Other:
- note added: "This is an example sheet. Make your own and add whatever you want!!"
- note removed: "This is an example sheet. Add whatever you want!"
Changed lines of the file:
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@@
 		)
 	)
-	(text "This is an example sheet. Add whatever you want!"
+	(text "This is an example sheet. Make your own and add whatever you want!!"
 		(exclude_from_sim no)
 		(at 146.05 23.622 0)
 		(effects
 			(font
-				(size 5.08 5.08)
+				(size 4.445 4.445)
 				(thickness 1.016)
 				(bold yes)
@@
 		(pts
 			(xy 127 100.33) (xy 163.83 100.33)
+		)
+		(stroke
+			(width 0)
+			(type default)
+		)
+	)
+	(polyline
+		(pts
+			(xy 144.78 118.11) (xy 144.78 161.29)
+		)
+		(stroke
+			(width 0)
+			(type default)
+		)
+	)
+	(polyline
+		(pts
+			(xy 134.62 137.16) (xy 153.67 137.16)
+		)
+		(stroke
+			(width 0)
+			(type default)
+		)
+	)
+	(polyline
+		(pts
+			(xy 123.19 182.88) (xy 144.78 161.29)
 		)
 		(stroke
@@
 		)
 		(stroke
+			(width 0)
+			(type default)
+		)
+	)
+	(polyline
+		(pts
+			(xy 144.78 161.29) (xy 166.37 182.88)
+		)
+		(stroke
